Commit message: Commit Repository of KUKA -KR150 - R2700-2 Variant

File: kuka_kr150_R2700_2_support/urdf/kuka_kr150_R2700_2_support.urdf (robot description, URDF)
Before this commit: robot urdf_assembly_v35, 9 links, 8 joints
Links:
- link base_link: geometry collision mesh filename=package://kuka_kr150_R2700_2_support/meshes/base_link.STL; visual mesh filename=package://kuka_kr150_R2700_2_support/meshes/base_link.STL
- link link_1: geometry collision mesh filename=package://kuka_kr150_R2700_2_support/meshes/link_1.STL; visual mesh filename=package://kuka_kr150_R2700_2_support/meshes/link_1.STL
- link link_2: geometry collision mesh filename=package://kuka_kr150_R2700_2_support/meshes/link_2.STL; visual mesh filename=package://kuka_kr150_R2700_2_support/meshes/link_2.STL
- link link_3: geometry collision mesh filename=package://kuka_kr150_R2700_2_support/meshes/link_3.STL; visual mesh filename=package://kuka_kr150_R2700_2_support/meshes/link_3.STL
- link link_4: geometry collision mesh filename=package://kuka_kr150_R2700_2_support/meshes/link_4.STL; visual mesh filename=package://kuka_kr150_R2700_2_support/meshes/link_4.STL
- link link_5: geometry collision mesh filename=package://kuka_kr150_R2700_2_support/meshes/link_5.STL; visual mesh filename=package://kuka_kr150_R2700_2_support/meshes/link_5.STL
- link link_6: geometry collision mesh filename=package://kuka_kr150_R2700_2_support/meshes/link_6.STL; visual mesh filename=package://kuka_kr150_R2700_2_support/meshes/link_6.STL
- link tool0: geometry collision mesh filename=package://kuka_kr150_R2700_2_support/meshes/tool0.STL; visual mesh filename=package://kuka_kr150_R2700_2_support/meshes/tool0.STL
