Commit message: Added KR4-Agilus variant and KUKA-RSI Support with Digital IO

File: kuka_kr10_support/urdf/kr10r1100sixx_macro.xacro (robot description, xacro)
@@ -1,6 +1,7 @@
 <?xml version="1.0"?>
 <robot xmlns:xacro="http://wiki.ros.org/xacro">
+  <xacro:include filename="$(find kuka_resources)/urdf/common_constants.xacro"/>
+  <xacro:include filename="$(find kuka_resources)/urdf/common_materials.xacro"/>
   <xacro:macro name="kuka_kr10r1100sixx" params="prefix">
-    <xacro:include filename="$(find kuka_resources)/urdf/common_materials.xacro"/>
     <link name="${prefix}base_link">
       <visual>
@@ -108,6 +109,6 @@
       </collision>
     </link>
-    <!-- Following REP199, this frame shall be use to attach EEF or other equipment -->
-    <link name="${prefix}flange" />
+    <!-- This frame corresponds to the $FLANGE coordinate system in KUKA KRC controllers. -->
+    <link name="${prefix}tool0"/>
     <joint name="${prefix}joint_a1" type="revolute">
       <origin xyz="0 0 0.400" rpy="0 0 0"/>
@@ -115,5 +116,5 @@
       <child link="${prefix}link_1"/>
       <axis xyz="0 0 -1"/>
-      <limit effort="0" lower="${radians(-170)}" upper="${radians(170)}" velocity="${radians(300)}"/>
+      <limit effort="0" lower="${-DEG2RAD * 170}" upper="${DEG2RAD * 170}" velocity="${DEG2RAD * 360}"/>
     </joint>
     <joint name="${prefix}joint_a2" type="revolute">
@@ -122,5 +123,5 @@
       <child link="${prefix}link_2"/>
       <axis xyz="0 1 0"/>
-      <limit effort="0" lower="${radians(-190)}" upper="${radians(45)}" velocity="${radians(225)}"/>
+      <limit effort="0" lower="${-DEG2RAD * 190}" upper="${DEG2RAD * 45}" velocity="${DEG2RAD * 300}"/>
     </joint>
     <joint name="${prefix}joint_a3" type="revolute">
@@ -129,5 +130,5 @@
       <child link="${prefix}link_3"/>
       <axis xyz="0 1 0"/>
-      <limit effort="0" lower="${radians(-120)}" upper="${radians(156)}" velocity="${radians(225)}"/>
+      <limit effort="0" lower="${-DEG2RAD * 120}" upper="${DEG2RAD * 156}" velocity="${DEG2RAD * 360}"/>
     </joint>
     <joint name="${prefix}joint_a4" type="revolute">
@@ -136,5 +137,5 @@
       <child link="${prefix}link_4"/>
       <axis xyz="-1 0 0"/>
-      <limit effort="0" lower="${radians(-185)}" upper="${radians(185)}" velocity="${radians(381)}"/>
+      <limit effort="0" lower="${-DEG2RAD * 185}" upper="${DEG2RAD * 185}" velocity="${DEG2RAD * 381}"/>
     </joint>
     <joint name="${prefix}joint_a5" type="revolute">
@@ -143,5 +144,5 @@
       <child link="${prefix}link_5"/>
       <axis xyz="0 1 0"/>
-      <limit effort="0" lower="${radians(-120)}" upper="${radians(120)}" velocity="${radians(311)}"/>
+      <limit effort="0" lower="${-DEG2RAD * 120}" upper="${DEG2RAD * 120}" velocity="${DEG2RAD * 388}"/>
     </joint>
     <joint name="${prefix}joint_a6" type="revolute">
@@ -150,10 +151,10 @@
       <child link="${prefix}link_6"/>
       <axis xyz="-1 0 0"/>
-      <limit effort="0" lower="${radians(-350)}" upper="${radians(350)}" velocity="${radians(492)}"/>
+      <limit effort="0" lower="${-DEG2RAD * 350}" upper="${DEG2RAD * 350}" velocity="${DEG2RAD * 615}"/>
     </joint>
-    <joint name="${prefix}joint_a6-flange" type="fixed">
+    <joint name="${prefix}joint_a6-tool0" type="fixed">
       <parent link="${prefix}link_6"/>
-      <child link="${prefix}flange"/>
-      <origin xyz="0 0 0" rpy="0 0 0"/>
+      <child link="${prefix}tool0"/>
+      <origin xyz="0 0 0" rpy="0 ${DEG2RAD * 90} 0"/>
     </joint>
     <!-- ROS base_link to KUKA $ROBROOT coordinate system transform -->
@@ -164,11 +165,4 @@
       <child link="${prefix}base"/>
     </joint>
-    <!-- This frame corresponds to the $TOOL coordinate system in KUKA KRC controllers -->
-    <link name="${prefix}tool0" />
-    <joint name="${prefix}flange-tool0" type="fixed">
-      <parent link="${prefix}flange"/>
-      <child link="${prefix}tool0"/>
-      <origin xyz="0 0 0" rpy="0 ${radians(90)} 0"/>
-    </joint>
   </xacro:macro>
 </robot>

File: kuka_kr120_support/urdf/kr120r2500pro_macro.xacro (robot description, xacro)
@@ -1,4 +1,5 @@
 <?xml version="1.0"?>
 <robot xmlns:xacro="http://wiki.ros.org/xacro">
+  <xacro:property name="DEG2RAD" value="0.017453292519943295"/>
   <xacro:macro name="kuka_kr120r2500pro" params="prefix">
     <!-- LINKS -->
@@ -143,6 +144,7 @@
       </collision>
     </link>
-    <!-- Following REP199, this frame shall be use to attach EEF or other equipment -->
-    <link name="${prefix}flange" />
+    <!-- tool 0 -->
+    <!-- This frame corresponds to the $FLANGE coordinate system in KUKA KRC controllers. -->
+    <link name="${prefix}tool0"/>
     <!-- END LINKS -->
     <!-- JOINTS -->
@@ -153,5 +155,5 @@
       <child link="${prefix}link_1"/>
       <axis xyz="0 0 -1"/>
-      <limit effort="0" lower="${-radians(185)}" upper="${radians(185)}" velocity="${radians(156)}"/>
+      <limit effort="0" lower="${-DEG2RAD * 185}" upper="${DEG2RAD * 185}" velocity="${DEG2RAD * 156}"/>
     </joint>
     <!-- joint 2 (A2) -->
@@ -161,5 +163,5 @@
       <child link="${prefix}link_2"/>
       <axis xyz="0 1 0"/>
-      <limit effort="0" lower="${-radians(155)}" upper="${radians(35)}" velocity="${radians(156)}"/>
+      <limit effort="0" lower="${-DEG2RAD * 155}" upper="${DEG2RAD * 35}" velocity="${DEG2RAD * 156}"/>
     </joint>
     <!-- joint 3 (A3) -->
@@ -169,5 +171,5 @@
       <child link="${prefix}link_3"/>
       <axis xyz="0 1 0"/>
-      <limit effort="0" lower="${-radians(130)}" upper="${radians(154)}" velocity="${radians(156)}"/>
+      <limit effort="0" lower="${-DEG2RAD * 130}" upper="${DEG2RAD * 154}" velocity="${DEG2RAD * 156}"/>
     </joint>
     <!-- joint 4 (A4) -->
@@ -177,5 +179,5 @@
       <child link="${prefix}link_4"/>
       <axis xyz="-1 0 0"/>
-      <limit effort="0" lower="${-radians(350)}" upper="${radians(350)}" velocity="${radians(330)}"/>
+      <limit effort="0" lower="${-DEG2RAD * 350}" upper="${DEG2RAD * 350}" velocity="${DEG2RAD * 330}"/>
     </joint>
     <!-- joint 5 (A5) -->
@@ -185,5 +187,5 @@
       <child link="${prefix}link_5"/>
       <axis xyz="0 1 0"/>
-      <limit effort="0" lower="${-radians(130)}" upper="${radians(130)}" velocity="${radians(330)}"/>
+      <limit effort="0" lower="${-DEG2RAD * 130}" upper="${DEG2RAD * 130}" velocity="${DEG2RAD * 330}"/>
     </joint>
     <!-- joint 6 (A6) -->
@@ -193,11 +195,11 @@
       <child link="${prefix}link_6"/>
       <axis xyz="-1 0 0"/>
-      <limit effort="0" lower="${-radians(350)}" upper="${radians(350)}" velocity="${radians(615)}"/>
+      <limit effort="0" lower="${-DEG2RAD * 350}" upper="${DEG2RAD * 350}" velocity="${DEG2RAD * 615}"/>
     </joint>
     <!-- tool frame - fixed frame -->
-    <joint name="${prefix}joint_a6-flange" type="fixed">
+    <joint name="${prefix}joint_a6-tool0" type="fixed">
       <parent link="${prefix}link_6"/>
-      <child link="${prefix}flange"/>
-      <origin xyz="0.215 0 0" rpy="0 0 0"/>
+      <child link="${prefix}tool0"/>
+      <origin xyz="0.215 0 0" rpy="0 ${DEG2RAD * 90} 0"/>
     </joint>
     <!-- END JOINTS -->
@@ -209,11 +211,4 @@
       <child link="${prefix}base"/>
     </joint>
-    <!-- This frame corresponds to the $TOOL coordinate system in KUKA KRC controllers -->
-    <link name="${prefix}tool0" />
-    <joint name="${prefix}flange-tool0" type="fixed">
-      <parent link="${prefix}flange"/>
-      <child link="${prefix}tool0"/>
-      <origin xyz="0 0 0" rpy="0 ${radians(90)} 0"/>
-    </joint>
   </xacro:macro>
 </robot>

File: kuka_kr150_support/urdf/kr150_2_macro.xacro (robot description, xacro)
@@ -109,6 +109,6 @@
     </link>
     <!-- tool link -->
-    <!-- This frame corresponds to the $TOOL coordinate system in KUKA KRC controllers. -->
-    <link name="${prefix}flange"/>
+    <!-- This frame corresponds to the $FLANGE coordinate system in KUKA KRC controllers. -->
+    <link name="${prefix}tool0"/>
     <!-- END LINKS -->
     <!-- JOINTS -->
@@ -162,8 +162,8 @@
     </joint>
     <!-- tool frame - fixed frame -->
-    <joint name="${prefix}joint_a6-flange" type="fixed">
+    <joint name="${prefix}joint_a6-tool0" type="fixed">
       <parent link="${prefix}link_6"/>
-      <child link="${prefix}flange"/>
-      <origin xyz="0 0 0" rpy="0 0 0"/>
+      <child link="${prefix}tool0"/>
+      <origin xyz="0 0 0" rpy="0 ${pi/2} 0"/>
     </joint>
     <!-- END JOINTS -->
@@ -171,14 +171,7 @@
     <link name="${prefix}base" />
     <joint name="${prefix}base_link-base" type="fixed">
-      <origin xyz="0 0 0" rpy="0 0 0"/>
-      <parent link="${prefix}base_link"/>
-      <child link="${prefix}base"/>
-    </joint>
-    <!-- This frame corresponds to the $TOOL coordinate system in KUKA KRC controllers -->
-    <link name="${prefix}tool0" />
-    <joint name="${prefix}flange-tool0" type="fixed">
-      <parent link="${prefix}flange"/>
-      <child link="${prefix}tool0"/>
-      <origin xyz="0 0 0" rpy="0 ${radians(90)} 0"/>
+      <origin xyz="0 0 0" rpy="0 0 0" />
+      <parent link="${prefix}base_link" />
+      <child link="${prefix}base" />
     </joint>
   </xacro:macro>

File: kuka_kr16_support/urdf/kr16_2_macro.xacro (robot description, xacro)
@@ -144,6 +144,6 @@
     </link>
     <!-- tool 0 -->
-    <!-- Following REP199, this frame shall be use to attach EEF or other equipment -->
-    <link name="${prefix}flange" />
+    <!-- This frame corresponds to the $FLANGE coordinate system in KUKA KRC controllers. -->
+    <link name="${prefix}tool0"/>
     <!-- END LINKS -->
     <!-- JOINTS -->
@@ -197,8 +197,8 @@
     </joint>
     <!-- tool frame - fixed frame -->
-    <joint name="${prefix}joint_a6-flange" type="fixed">
+    <joint name="${prefix}joint_a6-tool0" type="fixed">
       <parent link="${prefix}link_6"/>
-      <child link="${prefix}flange"/>
-      <origin xyz="0.158 0 0" rpy="0 0 0"/>
+      <child link="${prefix}tool0"/>
+      <origin xyz="0.158 0 0" rpy="0 ${radians(90)} 0"/>
     </joint>
     <!-- END JOINTS -->
@@ -210,11 +210,4 @@
       <child link="${prefix}base"/>
     </joint>
-    <!-- This frame corresponds to the $TOOL coordinate system in KUKA KRC controllers -->
-    <link name="${prefix}tool0" />
-    <joint name="${prefix}flange-tool0" type="fixed">
-      <parent link="${prefix}flange"/>
-      <child link="${prefix}tool0"/>
-      <origin xyz="0 0 0" rpy="0 ${radians(90)} 0"/>
-    </joint>
   </xacro:macro>
 </robot>

File: kuka_kr210_support/urdf/kr210l150_macro.xacro (robot description, xacro)
@@ -1,4 +1,7 @@
 <?xml version="1.0"?>
 <robot xmlns:xacro="http://wiki.ros.org/xacro">
+  <property name="pi" value="3.141592654"/>
+  <!--degrees to radians-->
+  <property name="deg" value="0.017453293"/>
   <xacro:macro name="kuka_kr210l150" params="prefix">
     <!-- links -->
@@ -10,5 +13,5 @@
       </inertial>
       <visual>
-        <origin xyz="0 0 0" rpy="${-radians(90)} 0 0"/>
+        <origin xyz="0 0 0" rpy="${-pi/2} 0 0"/>
         <geometry>
           <mesh filename="package://kuka_kr210_support/meshes/kr210l150/visual/base_link.dae"/>
@@ -19,5 +22,5 @@
       </visual>
       <collision>
-        <origin xyz="0 0 0" rpy="${-radians(90)} 0 0"/>
+        <origin xyz="0 0 0" rpy="${-pi/2} 0 0"/>
         <geometry>
           <mesh filename="package://kuka_kr210_support/meshes/kr210l150/collision/base_link.stl"/>
@@ -54,5 +57,5 @@
       </inertial>
       <visual>
-        <origin xyz="0 0 0" rpy="${-radians(90)} 0 0"/>
+        <origin xyz="0 0 0" rpy="${-pi/2} 0 0"/>
         <geometry>
           <mesh filename="package://kuka_kr210_support/meshes/kr210l150/visual/link_2.dae"/>
@@ -76,5 +79,5 @@
       </inertial>
       <visual>
-        <origin xyz="0 0 0" rpy="${-radians(90)} 0 0"/>
+        <origin xyz="0 0 0" rpy="${-pi/2} 0 0"/>
         <geometry>
           <mesh filename="package://kuka_kr210_support/meshes/kr210l150/visual/link_3.dae"/>
@@ -98,5 +101,5 @@
       </inertial>
       <visual>
-        <origin xyz="0 0 0" rpy="${-radians(90)} 0 0"/>
+        <origin xyz="0 0 0" rpy="${-pi/2} 0 0"/>
         <geometry>
           <mesh filename="package://kuka_kr210_support/meshes/kr210l150/visual/link_4.dae"/>
@@ -120,5 +123,5 @@
       </inertial>
       <visual>
-        <origin xyz="0 0 0" rpy="${-radians(90)} 0 0"/>
+        <origin xyz="0 0 0" rpy="${-pi/2} 0 0"/>
         <geometry>
           <mesh filename="package://kuka_kr210_support/meshes/kr210l150/visual/link_5.dae"/>
@@ -157,6 +160,6 @@
       </collision>
     </link>
-    <!-- This frame corresponds to the $TOOL coordinate system in KUKA KRC controllers. -->
-    <link name="${prefix}flange"/>
+    <!-- This frame corresponds to the $FLANGE coordinate system in KUKA KRC controllers. -->
+    <link name="${prefix}tool0"/>
     <!-- joints -->
     <joint name="${prefix}joint_a1" type="revolute">
@@ -165,5 +168,5 @@
       <child link="${prefix}link_1"/>
       <axis xyz="0 0 1"/>
-      <limit lower="${radians(-185)}" upper="${radians(185)}" effort="0" velocity="${radians(123)}"/>
+      <limit lower="${-185*deg}" upper="${185*deg}" effort="0" velocity="${123*deg}"/>
     </joint>
     <joint name="${prefix}joint_a2" type="revolute">
@@ -172,5 +175,5 @@
       <child link="${prefix}link_2"/>
       <axis xyz="0 1 0"/>
-      <limit lower="${radians(-45)}" upper="${radians(85)}" effort="0" velocity="${radians(115)}"/>
+      <limit lower="${-45*deg}" upper="${85*deg}" effort="0" velocity="${115*deg}"/>
     </joint>
     <joint name="${prefix}joint_a3" type="revolute">
@@ -179,5 +182,5 @@
       <child link="${prefix}link_3"/>
       <axis xyz="0 1 0"/>
-      <limit lower="${radians(-210)}" upper="${radians(65)}" effort="0" velocity="${radians(112)}"/>
+      <limit lower="${-210*deg}" upper="${(155-90)*deg}" effort="0" velocity="${112*deg}"/>
     </joint>
     <joint name="${prefix}joint_a4" type="revolute">
@@ -186,5 +189,5 @@
       <child link="${prefix}link_4"/>
       <axis xyz="1 0 0"/>
-      <limit lower="${radians(-350)}" upper="${radians(350)}" effort="0" velocity="${radians(179)}"/>
+      <limit lower="${-350*deg}" upper="${350*deg}" effort="0" velocity="${179*deg}"/>
     </joint>
     <joint name="${prefix}joint_a5" type="revolute">
@@ -193,5 +196,5 @@
       <child link="${prefix}link_5"/>
       <axis xyz="0 1 0"/>
-      <limit lower="${radians(-125)}" upper="${radians(125)}" effort="0" velocity="${radians(172)}"/>
+      <limit lower="${-125*deg}" upper="${125*deg}" effort="0" velocity="${172*deg}"/>
     </joint>
     <joint name="${prefix}joint_a6" type="revolute">
@@ -200,24 +203,10 @@
       <child link="${prefix}link_6"/>
       <axis xyz="1 0 0"/>
-      <limit lower="${radians(-350)}" upper="${radians(350)}" effort="0" velocity="${radians(219)}"/>
-    </joint>
-    <joint name="${prefix}link_6-flange" type="fixed">
+      <limit lower="${-350*deg}" upper="${350*deg}" effort="0" velocity="${219*deg}"/>
+    </joint>
+    <joint name="${prefix}link_6-tool0" type="fixed">
       <parent link="${prefix}link_6"/>
-      <child link="${prefix}flange"/>
+      <child link="${prefix}tool0"/>
       <origin xyz="0.0375 0 -0.00023924" rpy="0 0 0"/>
-    </joint>
-    <!-- ROS base_link to KUKA $ROBROOT coordinate system transform -->
-    <link name="${prefix}base" />
-    <joint name="${prefix}base_link-base" type="fixed">
-      <origin xyz="0 0 0" rpy="0 0 0"/>
-      <parent link="${prefix}base_link"/>
-      <child link="${prefix}base"/>
-    </joint>
-    <!-- This frame corresponds to the $TOOL coordinate system in KUKA KRC controllers -->
-    <link name="${prefix}tool0" />
-    <joint name="${prefix}flange-tool0" type="fixed">
-      <parent link="${prefix}flange"/>
-      <child link="${prefix}tool0"/>
-      <origin xyz="0 0 0" rpy="0 ${radians(90)} 0"/>
     </joint>
     <!-- rename 'Link1' to 'link_1', maintain bw-compatibility -->

File: kuka_kr3_support/urdf/kr3r540_macro.xacro (robot description, xacro)
@@ -108,8 +108,8 @@
       </collision>
     </link>
-    <!-- Following REP199, this frame shall be use to attach EEF or other equipment -->
-    <link name="${prefix}flange" />
+    <!-- This frame corresponds to the $FLANGE coordinate system in KUKA KRC controllers. -->
+    <link name="${prefix}tool0" />
     <joint name="${prefix}joint_a1" type="revolute">
-      <origin xyz="0 0 0.345" rpy="0 0 0"/>
+      <origin xyz="0 0 0.3z45" rpy="0 0 0"/>
       <parent link="${prefix}base_link"/>
       <child link="${prefix}link_1"/>
@@ -154,6 +154,6 @@
     <joint name="${prefix}joint_a6-tool0" type="fixed">
       <parent link="${prefix}link_6"/>
-      <child link="${prefix}flange"/>
-      <origin xyz="0 0 0" rpy="0 0 0"/>
+      <child link="${prefix}tool0"/>
+      <origin xyz="0 0 0" rpy="0 ${radians(90)} 0"/>
     </joint>
     <!-- ROS base_link to KUKA $ROBROOT coordinate system transform -->
@@ -164,11 +164,4 @@
       <child link="${prefix}base"/>
     </joint>
-    <!-- This frame corresponds to the $TOOL coordinate system in KUKA KRC controllers -->
-    <link name="${prefix}tool0" />
-    <joint name="${prefix}flange-tool0" type="fixed">
-      <parent link="${prefix}flange"/>
-      <child link="${prefix}tool0"/>
-      <origin xyz="0 0 0" rpy="0 ${radians(90)} 0"/>
-    </joint>
   </xacro:macro>
 </robot>

File: kuka_kr5_support/urdf/kr5_arc_macro.xacro (robot description, xacro)
@@ -205,11 +205,11 @@
     </link>
     <!-- tool link -->
-    <!-- Following REP199, this frame shall be use to attach EEF or other equipment -->
-    <link name="${prefix}flange" />
+    <!-- This frame corresponds to the $FLANGE coordinate system in KUKA KRC controllers. -->
+    <link name="${prefix}tool0"/>
     <!-- END LINKS -->
     <!-- JOINTS -->
     <!-- joint 1 (A1) -->
     <joint name="${prefix}joint_a1" type="revolute">
-      <origin xyz="0 0 0.4" rpy="${radians(180)} 0 0"/>
+      <origin xyz="0 0 0.4" rpy="${pi} 0 0"/>
       <parent link="${prefix}base_link"/>
       <child link="${prefix}link_1"/>
@@ -219,5 +219,5 @@
     <!-- joint 2 (A2) -->
     <joint name="${prefix}joint_a2" type="revolute">
-      <origin xyz="0.18 0 0" rpy="${radians(90)} 0 0"/>
+      <origin xyz="0.18 0 0" rpy="${pi/2} 0 0"/>
       <parent link="${prefix}link_1"/>
       <child link="${prefix}link_2"/>
@@ -235,5 +235,5 @@
     <!-- joint 4 (A4) -->
     <joint name="${prefix}joint_a4" type="revolute">
-      <origin xyz="0 -0.12 0" rpy="0 ${-radians(90)} 0"/>
+      <origin xyz="0 -0.12 0" rpy="0 ${-pi/2} 0"/>
       <parent link="${prefix}link_3"/>
       <child link="${prefix}link_4"/>
@@ -243,5 +243,5 @@
     <!-- joint 5 (A5) -->
     <joint name="${prefix}joint_a5" type="revolute">
-      <origin xyz="0 0 -0.62" rpy="0 ${radians(90)} 0"/>
+      <origin xyz="0 0 -0.62" rpy="0 ${pi/2} 0"/>
       <parent link="${prefix}link_4"/>
       <child link="${prefix}link_5"/>
@@ -251,5 +251,5 @@
     <!-- joint 6 (A6) -->
     <joint name="${prefix}joint_a6" type="revolute">
-      <origin xyz="0 0 0" rpy="0 ${-radians(90)} 0"/>
+      <origin xyz="0 0 0" rpy="0 ${-pi/2} 0"/>
       <parent link="${prefix}link_5"/>
       <child link="${prefix}link_6"/>
@@ -258,8 +258,8 @@
     </joint>
     <!-- tool frame - fixed frame -->
-    <joint name="${prefix}joint_a6-flange" type="fixed">
+    <joint name="${prefix}joint_a6-tool0" type="fixed">
       <parent link="${prefix}link_6"/>
-      <child link="${prefix}flange"/>
-      <origin xyz="0 0 -0.115" rpy="0 ${radians(90)} ${-radians(90)}"/>
+      <child link="${prefix}tool0"/>
+      <origin xyz="0 0 -0.115" rpy="0 ${-pi} ${-pi/2}"/>
     </joint>
     <!-- END JOINTS -->
@@ -267,14 +267,7 @@
     <link name="${prefix}base" />
     <joint name="${prefix}base_link-base" type="fixed">
-      <origin xyz="0 0 0" rpy="0 0 0"/>
-      <parent link="${prefix}base_link"/>
-      <child link="${prefix}base"/>
-    </joint>
-    <!-- This frame corresponds to the $TOOL coordinate system in KUKA KRC controllers -->
-    <link name="${prefix}tool0" />
-    <joint name="${prefix}flange-tool0" type="fixed">
-      <parent link="${prefix}flange"/>
-      <child link="${prefix}tool0"/>
-      <origin xyz="0 0 0" rpy="0 ${radians(90)} 0"/>
+      <origin xyz="0 0 0" rpy="0 0 0" />
+      <parent link="${prefix}base_link" />
+      <child link="${prefix}base" />
     </joint>
   </xacro:macro>
