Commit message: Added KR4-Agilus variant and KUKA-RSI Support with Digital IO

File: kuka_kr6_support/urdf/kr6r700sixx_macro.xacro (robot description, xacro)
@@ -1,16 +1,43 @@
 <?xml version="1.0"?>
 <robot xmlns:xacro="http://wiki.ros.org/xacro">
+  <!--xacro:include filename="$(find kuka_resources)/urdf/common_materials.xacro"/-->
+  <!--xacro:include filename="$(find kuka_kr6_gazebo)/urdf/kinect_v2.urdf.xacro" /-->
+  <xacro:macro name="default_inertial" params="mass">
+        <inertial>
+            <mass value="${mass}" />
+            <inertia ixx="1.0" ixy="0.0" ixz="0.0"
+                iyy="1.0" iyz="0.0"
+                izz="1.0" />
+        </inertial>
+    </xacro:macro>
   <xacro:include filename="$(find kuka_resources)/urdf/common_constants.xacro"/>
-  <xacro:include filename="$(find kuka_resources)/urdf/common_materials.xacro"/>
   <xacro:macro name="kuka_kr6r700sixx" params="prefix">
+<!--link name="${prefix}table">
+      <visual>
+	<origin xyz="-0.245 -0.645 0" rpy=" 0 0 ${pi/2}"/>
+        <geometry>
+          <mesh filename="package://kuka_kr6_support/meshes/kr6r700sixx/visual/Kinectnewsetupkukascene.stl" />
+        </geometry>
+        <material name="LightGrey">
+          <color rgba="0.7 0.7 0.7 1.0"/>
+        </material>
+      </visual>
+    </link-->
+  <!-- Kinect2 -->
+    <!--xacro:kinect_v2 parent="${prefix}base_link">
+      <origin xyz="0.332 -0.1425 1.312015" ryp="1.57 0 0"/>
+    </xacro:kinect_v2-->
     <link name="${prefix}base_link">
-      <visual>
+    <xacro:default_inertial mass="1"/>
+      <visual>
+        <!--origin xyz="0 0 0" rpy="0 0 0" /-->
         <origin xyz="0 0 0" rpy="0 0 0" />
         <geometry>
           <mesh filename="package://kuka_kr6_support/meshes/kr6_agilus/visual/base_link.dae" />
         </geometry>
-        <xacro:material_kuka_pedestal />
-      </visual>
-      <collision>
+        <!--xacro:material_kuka_pedestal /-->
+      </visual>
+      <collision>
+        <!--origin xyz="0 0 0" rpy="0 0 0" /-->
         <origin xyz="0 0 0" rpy="0 0 0" />
         <geometry>
@@ -20,4 +47,5 @@
     </link>
     <link name="${prefix}link_1">
+    <xacro:default_inertial mass="1"/>
       <visual>
         <origin xyz="0 0 0" rpy="0 0 0" />
@@ -25,5 +53,5 @@
           <mesh filename="package://kuka_kr6_support/meshes/kr6_agilus/visual/link_1.dae" />
         </geometry>
-        <xacro:material_kuka_orange />
+        <!--xacro:material_kuka_orange /-->
       </visual>
       <collision>
@@ -35,4 +63,5 @@
     </link>
     <link name="${prefix}link_2">
+    <xacro:default_inertial mass="1"/>
       <visual>
         <origin xyz="0 0 0" rpy="0 0 0" />
@@ -40,5 +69,5 @@
           <mesh filename="package://kuka_kr6_support/meshes/kr6r700sixx/visual/link_2.dae" />
         </geometry>
-        <xacro:material_kuka_orange />
+        <!--xacro:material_kuka_orange /-->
       </visual>
       <collision>
@@ -50,4 +79,5 @@
     </link>
     <link name="${prefix}link_3">
+    <xacro:default_inertial mass="1"/>
       <visual>
         <origin xyz="0 0 0" rpy="0 0 0" />
@@ -55,5 +85,5 @@
           <mesh filename="package://kuka_kr6_support/meshes/kr6_agilus/visual/link_3.dae" />
         </geometry>
-        <xacro:material_kuka_orange />
+        <!--xacro:material_kuka_orange /-->
       </visual>
       <collision>
@@ -65,4 +95,5 @@
     </link>
     <link name="${prefix}link_4">
+    <xacro:default_inertial mass="1"/>
       <visual>
         <origin xyz="0 0 0" rpy="0 0 0" />
@@ -70,5 +101,5 @@
           <mesh filename="package://kuka_kr6_support/meshes/kr6r700sixx/visual/link_4.dae" />
         </geometry>
-        <xacro:material_kuka_orange />
+        <!--xacro:material_kuka_orange /-->
       </visual>
       <collision>
@@ -80,4 +111,5 @@
     </link>
     <link name="${prefix}link_5">
+    <xacro:default_inertial mass="1"/>
       <visual>
         <origin xyz="0 0 0" rpy="0 0 0" />
@@ -85,5 +117,5 @@
           <mesh filename="package://kuka_kr6_support/meshes/kr6_agilus/visual/link_5.dae" />
         </geometry>
-        <xacro:material_kuka_orange />
+        <!--xacro:material_kuka_orange /-->
       </visual>
       <collision>
@@ -95,4 +127,5 @@
     </link>
     <link name="${prefix}link_6">
+    <xacro:default_inertial mass="1"/>
       <visual>
         <origin xyz="0 0 0" rpy="0 0 0" />
@@ -100,5 +133,5 @@
           <mesh filename="package://kuka_kr6_support/meshes/kr6_agilus/visual/link_6.dae" />
         </geometry>
-        <xacro:material_kuka_pedestal />
+        <!--xacro:material_kuka_pedestal /-->
       </visual>
       <collision>
@@ -109,12 +142,37 @@
       </collision>
     </link>
-    <!-- Following REP199, this frame shall be use to attach EEF or other equipment -->
-    <link name="${prefix}flange" />
-    <joint name="${prefix}joint_a1" type="revolute">
+<link name="${prefix}ee_link">
+      <visual>
+	<!--origin rpy="0 0 0" xyz=" -0.005 0.0045 -0.15"/-->
+<origin rpy="0 0 0" xyz="0 0 -0.07"/>
+        <geometry>
+<box size="0.10 0.06 0.15"/>
+          <!--mesh filename="package://kuka_kr6_support/meshes/kr6r700sixx/visual/gripneedle.stl" /-->
+        </geometry>
+        <material name="LightGrey">
+          <color rgba="0.7 0.7 0.7 1.0"/>
+        </material>
+      </visual>
+      <collision>
+        <geometry>
+          <box size="0.10 0.06 0.15"/>
+        </geometry>
+        <origin rpy="0 0 0" xyz="0 0 -0.07"/>
+      </collision>
+    </link>
+    <!-- This frame corresponds to the $FLANGE coordinate system in KUKA KRC controllers. -->
+    <link name="${prefix}tool0" />
+<!--joint name="${prefix}table_joint" type="fixed">
+      <origin xyz="0 0 -0.914" rpy="0 0 0"/>
+      <parent link="${prefix}base_link"/>
+      <child link="${prefix}table"/>
+    </joint-->
+<joint name="${prefix}joint_a1" type="revolute">
+<!--origin xyz="0 0 0.4" rpy="0 0 0"/-->
       <origin xyz="0 0 0.4" rpy="0 0 0"/>
       <parent link="${prefix}base_link"/>
       <child link="${prefix}link_1"/>
       <axis xyz="0 0 -1"/>
-      <limit lower="${radians(-170)}" upper="${radians(170)}" effort="0" velocity="${radians(360)}"/>
+      <limit lower="${-170 * DEG2RAD}" upper="${170 * DEG2RAD}" effort="0" velocity="${360 * DEG2RAD}"/>
     </joint>
     <joint name="${prefix}joint_a2" type="revolute">
@@ -123,5 +181,5 @@
       <child link="${prefix}link_2"/>
       <axis xyz="0 1 0"/>
-      <limit lower="${radians(-190)}" upper="${radians(45)}" effort="0" velocity="${radians(300)}"/>
+      <limit lower="${-190 * DEG2RAD}" upper="${45 * DEG2RAD}" effort="0" velocity="${300 * DEG2RAD}"/>
     </joint>
     <joint name="${prefix}joint_a3" type="revolute">
@@ -130,5 +188,5 @@
       <child link="${prefix}link_3"/>
       <axis xyz="0 1 0"/>
-      <limit lower="${radians(-120)}" upper="${radians(156)}" effort="0" velocity="${radians(360)}"/>
+      <limit lower="${-120 * DEG2RAD}" upper="${156 * DEG2RAD}" effort="0" velocity="${360 * DEG2RAD}"/>
     </joint>
     <joint name="${prefix}joint_a4" type="revolute">
@@ -137,5 +195,5 @@
       <child link="${prefix}link_4"/>
       <axis xyz="-1 0 0"/>
-      <limit lower="${radians(-185)}" upper="${radians(185)}" effort="0" velocity="${radians(381)}"/>
+      <limit lower="${-185 * DEG2RAD}" upper="${185 * DEG2RAD}" effort="0" velocity="${381 * DEG2RAD}"/>
     </joint>
     <joint name="${prefix}joint_a5" type="revolute">
@@ -144,5 +202,5 @@
       <child link="${prefix}link_5"/>
       <axis xyz="0 1 0"/>
-      <limit lower="${radians(-120)}" upper="${radians(120)}" effort="0" velocity="${radians(388)}"/>
+      <limit lower="${-120 * DEG2RAD}" upper="${120 * DEG2RAD}" effort="0" velocity="${388 * DEG2RAD}"/>
     </joint>
     <joint name="${prefix}joint_a6" type="revolute">
@@ -151,10 +209,16 @@
       <child link="${prefix}link_6"/>
       <axis xyz="-1 0 0"/>
-      <limit lower="${radians(-350)}" upper="${radians(350)}" effort="0" velocity="${radians(615)}"/>
-    </joint>
-    <joint name="${prefix}joint_a6-flange" type="fixed">
+      <limit lower="${-350 * DEG2RAD}" upper="${350 * DEG2RAD}" effort="0" velocity="${615 * DEG2RAD}"/>
+    </joint>
+ <joint name="${prefix}ee_fixed_joint" type="fixed">
+      <parent link="${prefix}link_6" />
+      <child link = "${prefix}ee_link" />
+      <origin xyz="0.15 0.0 0" rpy="0.0 ${90 * DEG2RAD} 0" />
+    </joint>
+    <joint name="${prefix}joint_a6-tool0" type="fixed">
       <parent link="${prefix}link_6"/>
-      <child link="${prefix}flange"/>
-      <origin xyz="0 0 0" rpy="0 0 0"/>
+      <child link="${prefix}tool0"/>
+      <!--origin xyz="0 0 0" rpy="0 ${90 * DEG2RAD} 0"/-->
+      <origin xyz="0.15 0 0" rpy="0 ${90 * DEG2RAD} 0"/>
     </joint>
     <!-- ROS base_link to KUKA $ROBROOT coordinate system transform -->
@@ -165,11 +229,4 @@
       <child link="${prefix}base"/>
     </joint>
-    <!-- This frame corresponds to the $TOOL coordinate system in KUKA KRC controllers -->
-    <link name="${prefix}tool0" />
-    <joint name="${prefix}flange-tool0" type="fixed">
-      <parent link="${prefix}flange"/>
-      <child link="${prefix}tool0"/>
-      <origin xyz="0 0 0" rpy="0 ${radians(90)} 0"/>
-    </joint>
   </xacro:macro>
 </robot>

File: kuka_kr6_support/urdf/kr6r900sixx_macro.xacro (robot description, xacro)
@@ -1,8 +1,16 @@
 <?xml version="1.0"?>
-<robot xmlns:xacro="http://wiki.ros.org/xacro">
+<robot xmlns:xacro="http://www.ros.org/wiki/xacro">
+    <xacro:macro name="default_inertial" params="mass">
+        <inertial>
+            <mass value="${mass}" />
+            <inertia ixx="1.0" ixy="0.0" ixz="0.0"
+                iyy="1.0" iyz="0.0"
+                izz="1.0" />
+        </inertial>
+    </xacro:macro>
   <xacro:include filename="$(find kuka_resources)/urdf/common_constants.xacro"/>
-  <xacro:include filename="$(find kuka_resources)/urdf/common_materials.xacro"/>
   <xacro:macro name="kuka_kr6r900sixx" params="prefix">
     <link name="${prefix}base_link">
+    <xacro:default_inertial mass="1"/>
       <visual>
         <origin xyz="0 0 0" rpy="0 0 0"/>
@@ -10,5 +18,4 @@
           <mesh filename="package://kuka_kr6_support/meshes/kr6_agilus/visual/base_link.dae" />
         </geometry>
-        <xacro:material_kuka_pedestal />
       </visual>
       <collision>
@@ -20,4 +27,5 @@
     </link>
     <link name="${prefix}link_1">
+    <xacro:default_inertial mass="1"/>
       <visual>
         <origin xyz="0 0 0" rpy="0 0 0"/>
@@ -25,5 +33,4 @@
           <mesh filename="package://kuka_kr6_support/meshes/kr6_agilus/visual/link_1.dae" />
         </geometry>
-        <xacro:material_kuka_orange />
       </visual>
       <collision>
@@ -35,4 +42,5 @@
     </link>
     <link name="${prefix}link_2">
+    <xacro:default_inertial mass="1"/>
       <visual>
         <origin xyz="0 0 0" rpy="0 0 0"/>
@@ -40,5 +48,4 @@
           <mesh filename="package://kuka_kr6_support/meshes/kr6r900sixx/visual/link_2.dae"/>
         </geometry>
-        <xacro:material_kuka_orange />
       </visual>
       <collision>
@@ -50,4 +57,5 @@
     </link>
     <link name="${prefix}link_3">
+    <xacro:default_inertial mass="1"/>
       <visual>
         <origin xyz="0 0 0" rpy="0 0 0"/>
@@ -55,5 +63,4 @@
           <mesh filename="package://kuka_kr6_support/meshes/kr6_agilus/visual/link_3.dae" />
         </geometry>
-        <xacro:material_kuka_orange />
       </visual>
       <collision>
@@ -65,4 +72,5 @@
     </link>
     <link name="${prefix}link_4">
+    <xacro:default_inertial mass="1"/>
       <visual>
         <origin xyz="0 0 0" rpy="0 0 0"/>
@@ -70,5 +78,4 @@
           <mesh filename="package://kuka_kr6_support/meshes/kr6r900sixx/visual/link_4.dae" />
         </geometry>
-        <xacro:material_kuka_orange />
       </visual>
       <collision>
@@ -80,4 +87,5 @@
     </link>
     <link name="${prefix}link_5">
+    <xacro:default_inertial mass="1"/>
       <visual>
         <origin xyz="0 0 0" rpy="0 0 0"/>
@@ -85,5 +93,4 @@
           <mesh filename="package://kuka_kr6_support/meshes/kr6_agilus/visual/link_5.dae" />
         </geometry>
-        <xacro:material_kuka_orange />
       </visual>
       <collision>
@@ -95,4 +102,5 @@
     </link>
     <link name="${prefix}link_6">
+    <xacro:default_inertial mass="1"/>
       <visual>
         <origin xyz="0 0 0" rpy="0 0 0"/>
@@ -100,5 +108,4 @@
           <mesh filename="package://kuka_kr6_support/meshes/kr6_agilus/visual/link_6.dae" />
         </geometry>
-        <xacro:material_kuka_pedestal />
       </visual>
       <collision>
@@ -109,6 +116,6 @@
       </collision>
     </link>
-    <!-- Following REP199, this frame shall be use to attach EEF or other equipment -->
-    <link name="${prefix}flange" />
+    <!-- This frame corresponds to the $FLANGE coordinate system in KUKA KRC controllers. -->
+    <link name="${prefix}tool0"/>
     <joint name="${prefix}joint_a1" type="revolute">
       <origin xyz="0 0 0.400" rpy="0 0 0"/>
@@ -116,5 +123,5 @@
       <child link="${prefix}link_1"/>
       <axis xyz="0 0 -1"/>
-      <limit effort="0" lower="${-radians(170)}" upper="${radians(170)}" velocity="${radians(360)}"/>
+      <limit effort="0" lower="${-DEG2RAD * 170}" upper="${DEG2RAD * 170}" velocity="${DEG2RAD * 360}"/>
     </joint>
     <joint name="${prefix}joint_a2" type="revolute">
@@ -123,5 +130,5 @@
       <child link="${prefix}link_2"/>
       <axis xyz="0 1 0"/>
-      <limit effort="0" lower="${-radians(190)}" upper="${radians(45)}" velocity="${radians(300)}"/>
+      <limit effort="0" lower="${-DEG2RAD * 190}" upper="${DEG2RAD * 45}" velocity="${DEG2RAD * 300}"/>
     </joint>
     <joint name="${prefix}joint_a3" type="revolute">
@@ -130,5 +137,5 @@
       <child link="${prefix}link_3"/>
       <axis xyz="0 1 0"/>
-      <limit effort="0" lower="${-radians(120)}" upper="${radians(156)}" velocity="${radians(360)}"/>
+      <limit effort="0" lower="${-DEG2RAD * 120}" upper="${DEG2RAD * 156}" velocity="${DEG2RAD * 360}"/>
     </joint>
     <joint name="${prefix}joint_a4" type="revolute">
@@ -137,5 +144,5 @@
       <child link="${prefix}link_4"/>
       <axis xyz="-1 0 0"/>
-      <limit effort="0" lower="${-radians(185)}" upper="${radians(185)}" velocity="${radians(381)}"/>
+      <limit effort="0" lower="${-DEG2RAD * 185}" upper="${DEG2RAD * 185}" velocity="${DEG2RAD * 381}"/>
     </joint>
     <joint name="${prefix}joint_a5" type="revolute">
@@ -144,5 +151,5 @@
       <child link="${prefix}link_5"/>
       <axis xyz="0 1 0"/>
-      <limit effort="0" lower="${-radians(120)}" upper="${radians(120)}" velocity="${radians(388)}"/>
+      <limit effort="0" lower="${-DEG2RAD * 120}" upper="${DEG2RAD * 120}" velocity="${DEG2RAD * 388}"/>
     </joint>
     <joint name="${prefix}joint_a6" type="revolute">
@@ -151,10 +158,10 @@
       <child link="${prefix}link_6"/>
       <axis xyz="-1 0 0"/>
-      <limit effort="0" lower="${-radians(350)}" upper="${radians(350)}" velocity="${radians(615)}"/>
+      <limit effort="0" lower="${-DEG2RAD * 350}" upper="${DEG2RAD * 350}" velocity="${DEG2RAD * 615}"/>
     </joint>
-    <joint name="${prefix}joint_a6-flange" type="fixed">
+    <joint name="${prefix}joint_a6-tool0" type="fixed">
       <parent link="${prefix}link_6"/>
-      <child link="${prefix}flange"/>
-      <origin xyz="0 0 0" rpy="0 0 0"/>
+      <child link="${prefix}tool0"/>
+      <origin xyz="0 0 0" rpy="0 ${DEG2RAD * 90} 0"/>
     </joint>
     <!-- ROS base_link to KUKA $ROBROOT coordinate system transform -->
@@ -165,11 +172,4 @@
       <child link="${prefix}base"/>
     </joint>
-    <!-- This frame corresponds to the $TOOL coordinate system in KUKA KRC controllers -->
-    <link name="${prefix}tool0" />
-    <joint name="${prefix}flange-tool0" type="fixed">
-      <parent link="${prefix}flange"/>
-      <child link="${prefix}tool0"/>
-      <origin xyz="0 0 0" rpy="0 ${radians(90)} 0"/>
-    </joint>
   </xacro:macro>
 </robot>

File: kuka_resources/urdf/common_colours.xacro (robot description, xacro)
@@ -72,9 +72,5 @@
   <!-- RAL 9002 - gray white  -->
   <xacro:property name="colour_kuka_ral_gray_white"       value="${215/255} ${213/255} ${203/255} 1.0" />
-  <!-- RAL 9007 - grey aluminium -->
-  <xacro:property name="colour_kuka_ral_gray_aluminium"   value="${135/255} ${133/255} ${129/255} 1.0" />
   <!-- RAL 9010 - pure white  -->
   <xacro:property name="colour_kuka_ral_pure_white"       value="${241/255} ${236/255} ${255/255} 1.0" />
-  <!-- RAL 9016 - traffic white -->
-  <xacro:property name="colour_kuka_ral_traffic_white"    value="${241/255}  ${240/255} ${234/255} 1.0" />
 </robot>

File: kuka_resources/urdf/common_materials.xacro (robot description, xacro)
@@ -152,9 +152,4 @@
     </material>
   </xacro:macro>
-  <xacro:macro name="material_kuka_ral_gray_aluminium">
-    <material name="">
-      <color rgba="${colour_kuka_ral_gray_aluminium}"/>
-    </material>
-  </xacro:macro>
   <xacro:macro name="material_kuka_ral_pure_white">
     <material name="">
@@ -162,8 +157,3 @@
     </material>
   </xacro:macro>
-  <xacro:macro name="material_kuka_ral_traffic_white">
-    <material name="">
-      <color rgba="${colour_kuka_ral_traffic_white}"/>
-    </material>
-  </xacro:macro>
 </robot>
